File: usbhs_v0.3.kicad_pcb (KiCad board)
At the start: 4 copper layers, 68.5 x 30 mm, 66 parts, among them J1 USB_B, J2 Conn_01x02, J3 Conn_01x03, J4 Conn_02x10_Top_Bottom, SW1 SW_Push, SW2 SW_Push, U1 SY8088, U2 USBLC6-2SC6, U3 STM32F446RETx, U4 USB3300-EZK, U5 74LVC1G3157, Y1 12.288M

Commit message: modified:   .gitignore 	modified:   usbhs_v0.3.kicad_pcb 	modified:   usbhs_v0.3.kicad_sch 	new file:   usbhs_v0.3.xml
Parts:
- R10, R18, R19, R5: value 10k -> 1k
Changed lines of the file:
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@@
       (layerselection 0x00010fc_ffffffff)
       (disableapertmacros false)
-      (usegerberextensions false)
-      (usegerberattributes true)
-      (usegerberadvancedattributes true)
-      (creategerberjobfile true)
+      (usegerberextensions true)
+      (usegerberattributes false)
+      (usegerberadvancedattributes false)
+      (creategerberjobfile false)
       (svguseinch false)
       (svgprecision 6)
@@
       (psa4output false)
       (plotreference true)
-      (plotvalue true)
+      (plotvalue false)
       (plotinvisibletext false)
       (sketchpadsonfab false)
-      (subtractmaskfromsilk false)
+      (subtractmaskfromsilk true)
       (outputformat 1)
       (mirror false)
-      (drillshape 1)
+      (drillshape 0)
       (scaleselection 1)
-      (outputdirectory "")
+      (outputdirectory "gbr/")
     )
   )
@@
     (fp_line (start 1.6 0.8) (end -1.6 0.8) (layer "F.Fab") (width 0.1))
     (fp_line (start -1.6 0.8) (end -1.6 -0.8) (layer "F.Fab") (width 0.1))
-    (pad "1" smd roundrect (at -1.475 0 270) (size 1.15 1.8) (layers "F.Cu" "F.Paste" "F.Mask") (roundrect_rratio 0.217391)
+    (pad "1" smd roundrect (at -1.475 0 270) (size 1.15 1.8) (layers "F.Cu" "F.Paste" "F.Mask") (roundrect_rratio 0.2173913043)
       (net 3 "+3V3") (pintype "passive"))
-    (pad "2" smd roundrect (at 1.475 0 270) (size 1.15 1.8) (layers "F.Cu" "F.Paste" "F.Mask") (roundrect_rratio 0.217391)
+    (pad "2" smd roundrect (at 1.475 0 270) (size 1.15 1.8) (layers "F.Cu" "F.Paste" "F.Mask") (roundrect_rratio 0.2173913043)
       (net 2 "GND") (pintype "passive"))
     (model "${KICAD6_3DMODEL_DIR}/Capacitor_SMD.3dshapes/C_1206_3216Metric.wrl"
@@
       (effects (font (size 1 1) (thickness 0.15)))
     )
-    (fp_text value "10k" (at 0 1.43) (layer "F.Fab")
+    (fp_text value "1k" (at 0 1.43) (layer "F.Fab")
       (effects (font (size 1 1) (thickness 0.15)))
     )
@@
       (effects (font (size 1 1) (thickness 0.15)))
     )
-    (fp_text value "10k" (at 0 1.43) (layer "F.Fab")
+    (fp_text value "1k" (at 0 1.43) (layer "F.Fab")
       (effects (font (size 1 1) (thickness 0.15)))
     )
@@
     (fp_line (start 1.6 -0.8) (end 1.6 0.8) (layer "F.Fab") (width 0.1))
     (fp_line (start -1.6 -0.8) (end 1.6 -0.8) (layer "F.Fab") (width 0.1))
-    (pad "1" smd roundrect (at -1.475 0) (size 1.15 1.8) (layers "F.Cu" "F.Paste" "F.Mask") (roundrect_rratio 0.217391)
+    (pad "1" smd roundrect (at -1.475 0) (size 1.15 1.8) (layers "F.Cu" "F.Paste" "F.Mask") (roundrect_rratio 0.2173913043)
       (net 65 "/USB_SHIELD") (pintype "passive"))
-    (pad "2" smd roundrect (at 1.475 0) (size 1.15 1.8) (layers "F.Cu" "F.Paste" "F.Mask") (roundrect_rratio 0.217391)
+    (pad "2" smd roundrect (at 1.475 0) (size 1.15 1.8) (layers "F.Cu" "F.Paste" "F.Mask") (roundrect_rratio 0.2173913043)
       (net 2 "GND") (pintype "passive"))
     (model "${KICAD6_3DMODEL_DIR}/Capacitor_SMD.3dshapes/C_1206_3216Metric.wrl"
@@
     (fp_line (start -1.6 0.8) (end -1.6 -0.8) (layer "F.Fab") (width 0.1))
     (fp_line (start -1.6 -0.8) (end 1.6 -0.8) (layer "F.Fab") (width 0.1))
-    (pad "1" smd roundrect (at -1.475 0 270) (size 1.15 1.8) (layers "F.Cu" "F.Paste" "F.Mask") (roundrect_rratio 0.217391)
+    (pad "1" smd roundrect (at -1.475 0 270) (size 1.15 1.8) (layers "F.Cu" "F.Paste" "F.Mask") (roundrect_rratio 0.2173913043)
       (net 1 "VBUS") (pintype "passive"))
-    (pad "2" smd roundrect (at 1.475 0 270) (size 1.15 1.8) (layers "F.Cu" "F.Paste" "F.Mask") (roundrect_rratio 0.217391)
+    (pad "2" smd roundrect (at 1.475 0 270) (size 1.15 1.8) (layers "F.Cu" "F.Paste" "F.Mask") (roundrect_rratio 0.2173913043)
       (net 2 "GND") (pintype "passive"))
     (model "${KICAD6_3DMODEL_DIR}/Capacitor_SMD.3dshapes/C_1206_3216Metric.wrl"
@@
       (effects (font (size 1 1) (thickness 0.15)))
     )
-    (fp_text value "10k" (at 0 1.43) (layer "F.Fab")
+    (fp_text value "1k" (at 0 1.43) (layer "F.Fab")
       (effects (font (size 1 1) (thickness 0.15)))
     )
@@
       (effects (font (size 1 1) (thickness 0.15)))
     )
-    (fp_text value "10k" (at 0 1.43) (layer "F.Fab")
+    (fp_text value "1k" (at 0 1.43) (layer "F.Fab")
       (effects (font (size 1 1) (thickness 0.15)))
     )
@@
     )
   )
-  (footprint "Symbol:OSHW-Logo2_7.3x6mm_SilkScreen" (layer "F.Cu")
+  (footprint "Symbol:OSHW-Logo2_7.3x6mm_SilkScreen" locked (layer "F.Cu")
     (at 75 67)
     (descr "Open Source Hardware Symbol")
@@
         (xy 60.25 53.5)
         (xy 60.25 57.75)
-        (xy 60.25 57.75)
-        (xy 58.5 59.5)
         (xy 58.5 59.5)
         (xy 57.25 60.75)

Commit message: modified:   .gitignore 	modified:   usbhs_v0.3.kicad_pcb 	modified:   usbhs_v0.3.kicad_sch 	deleted:    usbhs_v0.3.xml
Parts:
- removed the C13 at (89.0, 56.0)
- removed the C9 at (95.0, 56.0)
- removed Y1: 12.288M, Crystal:Crystal_SMD_3225-4Pin_3.2x2.5mm
- added C12: 103, Capacitor_SMD:C_0603_1608Metric, F.Cu at (95.0, 55.8)
- added FB1: 600R, Inductor_SMD:L_0603_1608Metric, F.Cu at (94.2, 53.2)
- added X1: 24.576M, Crystal:Crystal_SMD_3225-4Pin_3.2x2.5mm, F.Cu at (92.0, 55.8)
- D1: value LED -> LED_WHITE
- D2: value LED -> LED_BLUE
- D3: value LED -> LED_RED
- D4: value LED -> LED_GREEN
- D5: value LED -> LED_YELLOW
- R21: value 10k -> 1k
- renumbered C11 to C10, C12 to C11, C14 to C13, C15 to C14, C16 to C15, C17 to C16, C18 to C17, C10 to C9
Connections:
- U3 pad 6: Net-(C13-Pad1) -> unconnected-(U3-Pad6)
Routing:
- net Net-(C12-Pad2): track 0.00 -> 5.43 mm
- net Net-(C13-Pad1): track 4.70 -> 0.00 mm
- net Net-(U3-Pad5): track 6.94 -> 3.08 mm
- net GND: track 34.2 -> 31.5 mm, vias 74 -> 61
- net +3V3: track 132.8 -> 133.5 mm, vias 23 -> 24
- added copper zone on F.Cu, net Net-(C12-Pad2)

Commit message: modified:   usbhs_v0.3.kicad_pcb 	modified:   usbhs_v0.3.kicad_sch
Parts:
- added R8: 0, Resistor_SMD:R_0603_1608Metric, F.Cu at (99.8, 67.2)
- renumbered R9 to R10, R10 to R11, R11 to R12, R12 to R13, R13 to R14, R14 to R15, R15 to R16, R16 to R17, R17 to R18, R18 to R19, R19 to R20, R20 to R21, R21 to R22, R22 to R23, R8 to R9
Connections:
- U3 pad 54: unconnected-(U3-Pad54) -> /EXTI2
- U3 pad 61: unconnected-(U3-Pad61) -> /MUTE
Routing:
- net /MUTE: track 0.00 -> 16.2 mm, vias 0 -> 2
- net /EXTI2: track 0.00 -> 5.16 mm, vias 0 -> 2
- net /I2S3_WS: track 6.22 -> 10.0 mm
- net /I2S3_CK: track 13.7 -> 14.8 mm, vias 0 -> 2

Commit message: modified:   img.png 	modified:   usbhs_v0.3.kicad_pcb 	modified:   usbhs_v0.3.kicad_prl 	modified:   usbhs_v0.3.kicad_pro 	modified:   usbhs_v0.3.kicad_sch 	new file:   usbhs_v0.3.kicad_sch-bak
Parts:
- removed the C1 at (63.5, 73.0)
- removed the C12 at (95.0, 55.8)
- removed the D3 at (78.5, 78.0)
- removed D4: LED_GREEN, LED_SMD:LED_0603_1608Metric
- removed FB1: 600R, Inductor_SMD:L_0603_1608Metric
- removed the J2 at (83.0, 53.0)
- removed J4: Conn_02x10_Top_Bottom, Connector_PinHeader_2.54mm:PinHeader_2x10_P2.54mm_Vertical
- removed the JP1 at (113.8, 63.8)
- removed the R11 at (86.5, 76.5)
- removed the R19 at (78.5, 76.5)
- removed the R20 at (82.5, 76.5)
- removed the R21 at (105.0, 71.2)
- removed X1: 24.576M, Crystal:Crystal_SMD_3225-4Pin_3.2x2.5mm
- added C13: 33p, Capacitor_SMD:C_0603_1608Metric, F.Cu at (94.0, 54.0)
- added C14: 33p, Capacitor_SMD:C_0603_1608Metric, F.Cu at (78.5, 54.0)
- added C16: 104, Capacitor_SMD:C_0402_1005Metric, F.Cu at (77.2, 65.2)
- added C17: 104, Capacitor_SMD:C_0402_1005Metric, F.Cu at (77.2, 60.2)
- added C18: 104, Capacitor_SMD:C_0402_1005Metric, F.Cu at (71.2, 57.8)
- added C21: 475, Capacitor_SMD:C_0603_1608Metric, F.Cu at (74.8, 57.2)
- added C5: 104, Capacitor_SMD:C_0402_1005Metric, F.Cu at (94.5, 57.5)
- added C9: 22p, Capacitor_SMD:C_0603_1608Metric, F.Cu at (70.2, 78.0)
- added J3: Conn_02x10_Odd_Even, Connector_PinHeader_2.54mm:PinHeader_2x10_P2.54mm_Vertical, F.Cu at (111.0, 77.0)
- added R4: 150k, Resistor_SMD:R_0603_1608Metric, F.Cu at (64.2, 78.0)
- added R7: 1k, Resistor_SMD:R_0603_1608Metric, F.Cu at (57.8, 76.2)
- added R9: 10, Resistor_SMD:R_0603_1608Metric, F.Cu at (105.0, 73.8)
- added Y1: 12.288M, Crystal:Crystal_SMD_HC49-SD, F.Cu at (86.2, 54.0)
- C1: renamed from C2; footprint Capacitor_SMD:C_0603_1608Metric -> Capacitor_SMD:C_0402_1005Metric
- C10: renamed from C9; footprint Capacitor_SMD:C_0603_1608Metric -> Capacitor_SMD:C_0402_1005Metric
- C11: renamed from C10; value 104 -> 104/50V
- C12: renamed from C11; footprint Capacitor_SMD:C_0603_1608Metric -> Capacitor_SMD:C_0402_1005Metric
- C15: renamed from C13; footprint Capacitor_SMD:C_0603_1608Metric -> Capacitor_SMD:C_0402_1005Metric
- C19: renamed from C14; footprint Capacitor_SMD:C_0603_1608Metric -> Capacitor_SMD:C_0402_1005Metric
- C2: renamed from C3; footprint Capacitor_SMD:C_0603_1608Metric -> Capacitor_SMD:C_0402_1005Metric
- C23: renamed from C17; value 103 -> 104; footprint Capacitor_SMD:C_0603_1608Metric -> Capacitor_SMD:C_0402_1005Metric
- C3: renamed from C4; footprint Capacitor_SMD:C_0603_1608Metric -> Capacitor_SMD:C_0402_1005Metric
- C4: renamed from C5; footprint Capacitor_SMD:C_0603_1608Metric -> Capacitor_SMD:C_0402_1005Metric
- C6: footprint Capacitor_SMD:C_0603_1608Metric -> Capacitor_SMD:C_0402_1005Metric
- C7: value 106/50V -> 106
- C8: value 10p -> 106; footprint Capacitor_SMD:C_0603_1608Metric -> Capacitor_SMD:C_1206_3216Metric
- D1: value LED_WHITE -> LED_Dual_KAK; footprint LED_SMD:LED_0603_1608Metric -> LED_THT:LED_D3.0mm-3
- D2: value LED_BLUE -> LED_WHITE
- JP1: renamed from JP2; moved to F.Cu
- R1: value 453k -> 1k
- R2: value 22 -> 1k
- R3: value 100k -> 680k
- R5: value 1k -> 0
- moved R5 44.4 mm to (99.5, 59.5)
- moved D2 28.8 mm to (57.8, 78.0), turned to 0 degrees
- moved D1 23.5 mm to (82.0, 77.2), turned to 0 degrees
- moved R8 20.9 mm to (77.5, 58.0), turned to 180 degrees
- moved R2 17.8 mm to (87.8, 73.8), turned to 180 degrees
- moved R1 16.5 mm to (84.8, 73.8)
- moved C20 14.9 mm to (76.5, 67.0), turned to 180 degrees
- moved D3 11.3 mm to (114.5, 60.2)
- moved R15 10.8 mm to (104.2, 76.2)
- moved R16 10.8 mm to (105.8, 76.2)
- moved JP1 9.29 mm to (114.2, 57.7)
- moved R21 8.27 mm to (114.5, 61.8)
- moved C15 7.29 mm to (67.8, 61.8), turned to 180 degrees
- moved REF** 6.97 mm to (76.8, 73.8)
- moved C8 6.17 mm to (63.2, 74.8), turned to 90 degrees
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- renumbered C15 to C20, C16 to C22, D5 to D3, J3 to J2, R7 to R10, R8 to R11, R9 to R12, R10 to R13, R12 to R14, R13 to R15, R14 to R16, R15 to R17, R16 to R18, R17 to R19, R18 to R20, R22 to R21, R23 to R22, R4 to R6, R6 to R8
Connections:
- C15 pad 1: GND -> +3V3
- C15 pad 2: +3V3 -> GND
- C20 pad 2: Net-(C15-Pad2) -> Net-(C20-Pad2)
- C7 pad 1: +3V3 -> GND
- C7 pad 2: GND -> +3V3
- C8 pad 1: Net-(C8-Pad1) -> GND
- C8 pad 2: +3V3 -> VBUS
- D1 pad 1: GND -> Net-(D1-Pad1)
- D1 pad 2: Net-(D1-Pad2) -> +3V3
- D2 pad 2: Net-(D2-Pad2) -> +3V3
- R1 pad 1: Net-(C8-Pad1) -> Net-(D1-Pad1)
- R1 pad 2: +3V3 -> /LED1
- R2 pad 1: Net-(R2-Pad1) -> Net-(D1-Pad3)
- R2 pad 2: /UART4_TX -> /LED2
- R3 pad 1: GND -> +3V3
- R3 pad 2: Net-(C8-Pad1) -> Net-(C9-Pad2)
- R5 pad 1: Net-(D1-Pad2) -> /I2S1_WS
- R5 pad 2: +3V3 -> /I2S3_WS
- U1 pad 5: Net-(C8-Pad1) -> Net-(C9-Pad2)
- U3 pad 14: Net-(R2-Pad1) -> unconnected-(U3-Pad14)
- U3 pad 2: unconnected-(U3-Pad2) -> /F1
- U3 pad 20: unconnected-(U3-Pad20) -> /I2S1_WS
- U3 pad 3: unconnected-(U3-Pad3) -> /F2
- U3 pad 37: Net-(D2-Pad1) -> unconnected-(U3-Pad37)
- U3 pad 4: unconnected-(U3-Pad4) -> /F3
- U3 pad 42: unconnected-(U3-Pad42) -> Net-(R9-Pad1)
- U3 pad 45: unconnected-(U3-Pad45) -> /PDN
- U3 pad 52: /DSDOE -> unconnected-(U3-Pad52)
- U3 pad 56: unconnected-(U3-Pad56) -> /DSDOE
- U3 pad 6: unconnected-(U3-Pad6) -> Net-(C14-Pad1)
- U3 pad 61: /MUTE -> unconnected-(U3-Pad61)
- U3 pad 62: unconnected-(U3-Pad62) -> /F0
- U4 pad 15: Net-(C15-Pad2) -> Net-(C20-Pad2)
- U4 pad 26: Net-(C15-Pad2) -> Net-(C21-Pad2)
- U5 pad 4: Net-(R21-Pad1) -> /I2S_LRCK/DSD2
Routing:
- net +3V3: track 133.5 -> 184.4 mm, vias 24 -> 22
- net /24M_CK: track 47.3 -> 6.46 mm, vias 2 -> 0
- net /PDN: track 0.00 -> 27.4 mm, vias 0 -> 1
- net /I2C1_SDA: track 13.3 -> 37.6 mm
- net /F1: track 0.00 -> 21.3 mm
- net /F3: track 0.00 -> 20.6 mm
- net /F2: track 0.00 -> 20.5 mm
- net /I2S_MCK: track 20.2 -> 40.4 mm, vias 0 -> 2
- net /RCC_MCO1: track 2.81 -> 22.0 mm, vias 0 -> 2
- net Net-(C14-Pad1): track 0.00 -> 17.4 mm
- net /I2S1_WS: track 0.00 -> 17.1 mm, vias 0 -> 4
- net Net-(R9-Pad1): track 0.00 -> 16.2 mm
- net /MUTE: track 16.2 -> 0.00 mm, vias 2 -> 0
- net Net-(C15-Pad2): track 14.9 -> 0.00 mm, vias 2 -> 0
- net /F0: track 0.00 -> 13.0 mm
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- added copper zone on B.Cu, net +3V3
- added copper zone on B.Cu, net /USB_SHIELD
- removed copper zone on In2.Cu, net +3V3
- removed copper zone on In1.Cu, net GND
- removed copper zone on In2.Cu, net GND
- removed copper zone on F.Cu, net Net-(C12-Pad2) (its old number)
Other:
- copper layers 4 -> 2
- board text added: "2023/05 v0.31"
- board text added: "3V3"
- board text added: "5V"
- board text added: "BCK"
- board text added: "DATA"
- board text added: "DSDOE"
- board text added: "F0"
- board text added: "F1"
- board text added: "F2"
- board text added: "F3"
- board text added: "LRCK"
- board text added: "MCLK"
- board text added: "NC"
- board text added: "SCL"
- board text added: "SDA"
- board text added: "SPDIF_TX"
- board text removed: "TX"
